Commit message: Replaced hard-coded file path.

File: human_robot_gym/models/assets/robots/schunk/robot_pybullet.urdf (robot description, URDF)
Before this commit: robot schunk_lwa4p, 9 links, 8 joints
Links:
- link arm_podest_link: geometry collision mesh filename=package://schunk/meshes/arm_base_link.stl; visual mesh filename=package://schunk/meshes/arm_base_link.stl
