Commit message: Requirements

File: human_robot_gym/models/assets/robots/schunk/robot.urdf (robot description, URDF)
Before this commit: robot schunk_lwa4p, 11 links, 10 joints
Links:
- link end: geometry collision cylinder length=0.000001 radius=0.07; visual cylinder length=0.000001 radius=0.1
- link gripper: geometry collision cylinder length=0.15 radius=0.07; visual cylinder length=0.15 radius=0.07
Joints:
- joint end_joint: origin xyz=0 0 0.05 rpy=0 0 0 -> xyz=0 0 0.075 rpy=0 0 0
- joint fixed_gripper_joint: origin xyz=0 0 0.12 rpy=0 0 0 -> xyz=0 0 0.17 rpy=0 0 0

Commit message: Fixed observations

File: human_robot_gym/models/assets/robots/schunk/robot.urdf (robot description, URDF)
Before this commit: robot schunk_lwa4p, 11 links, 10 joints
Links:
- link end: geometry collision cylinder length=0.000001 radius=0.07; visual cylinder length=0.000001 radius=0.07

Commit message: Changed the way self collision is computed to speed up simulation by 30%.

File: human_robot_gym/models/assets/robots/schunk/robot.urdf (robot description, URDF)
Before this commit: robot schunk_lwa4p, 11 links, 10 joints
Links:
- link end: geometry collision cylinder length=0.000001 radius=0.05; visual cylinder length=0.000001 radius=0.05
- link gripper: geometry collision cylinder length=0.14 radius=0.07; visual cylinder length=0.14 radius=0.07
Joints:
- joint end_joint: origin xyz=0 0 0.075 rpy=0 0 0 -> xyz=0 0 0.065 rpy=0 0 0
- joint fixed_gripper_joint: origin xyz=0 0 0.17 rpy=0 0 0 -> xyz=0 0 0.16 rpy=0 0 0

Commit message: Manually changed robot.urdf

File: human_robot_gym/models/assets/robots/schunk/robot.urdf (robot description, URDF)
Before this commit: robot schunk_lwa4p, 11 links, 10 joints
Links:
- link gripper: geometry collision cylinder length=0.1 radius=0.07; visual cylinder length=0.1 radius=0.07
Joints:
- joint end_joint: origin xyz=0 0 0.065 rpy=0 0 0 -> xyz=0 0 0.045 rpy=0 0 0

Commit message: robot.urdf fine tuning

File: human_robot_gym/models/assets/robots/schunk/robot.urdf (robot description, URDF)
Before this commit: robot schunk_lwa4p, 11 links, 10 joints
Links:
- link gripper: geometry collision cylinder length=0.11 radius=0.07; visual cylinder length=0.11 radius=0.07
Joints:
- joint end_joint: origin xyz=0 0 0.045 rpy=0 0 0 -> xyz=0 0 0.035 rpy=0 0 0
