Commit message: Kinova3 New URDF - all revolute joints

File: human_robot_gym/models/assets/robots/kinova3/kinova3.urdf (robot description, URDF)
Before this commit: robot GEN3_URDF_V12, 9 links, 8 joints
Joints:
- joint Actuator7: type continuous -> revolute
- joint EndEffector: limit (none) -> lower=-3.14 upper=3.14 effort=9.0 velocity=0.8727; type fixed -> revolute
